Commit message: Improve simulator responsiveness and correct preplaced goal contacts
Release 0.1.6 with explicit workspace builds, scene reuse, lazy GPU replay visuals, configurable PhysX CPU workers, and the academic/noncommercial license. Preserve fixed-step execution and document native validation limits.

File: assets/objects/pin_blue_red.urdf (robot description, URDF)
Before this commit: robot override_pin_blue_red, 1 links, 0 joints
Links:
- link pin: geometry collision mesh filename=pin_flange.stl; collision mesh filename=pin_root_-1_band_0.stl

File: assets/objects/pin_blue_yellow.urdf (robot description, URDF)
Before this commit: robot override_pin_blue_yellow, 1 links, 0 joints
Links:
- link pin: geometry collision mesh filename=pin_flange.stl; collision mesh filename=pin_root_-1_band_0.stl

File: assets/objects/pin_red_blue.urdf (robot description, URDF)
Before this commit: robot override_pin_red_blue, 1 links, 0 joints
Links:
- link pin: geometry collision mesh filename=pin_flange.stl; collision mesh filename=pin_root_-1_band_0.stl

File: assets/objects/pin_red_yellow.urdf (robot description, URDF)
Before this commit: robot override_pin_red_yellow, 1 links, 0 joints
Links:
- link pin: geometry collision mesh filename=pin_flange.stl; collision mesh filename=pin_root_-1_band_0.stl

File: assets/objects/pin_yellow_yellow.urdf (robot description, URDF)
Before this commit: robot override_pin_yellow_yellow, 1 links, 0 joints
Links:
- link pin: geometry collision mesh filename=pin_flange.stl; collision mesh filename=pin_root_-1_band_0.stl
